Commit message: minor changes

File: scout/scout_description/urdf/gen3_macro.xacro (robot description, xacro)
@@ -22,5 +22,5 @@
     gripper_max_force:=100.0
     use_fake_hardware:=false
-    fake_sensor_commands:=false
+    mock_sensor_commands:=false
     sim_gazebo:=false
     sim_ignition:=false
@@ -35,5 +35,5 @@
       name="${prefix}KortexMultiInterfaceHardware" prefix="${prefix}"
       use_fake_hardware="${use_fake_hardware}"
-      fake_sensor_commands="${fake_sensor_commands}"
+      mock_sensor_commands="${mock_sensor_commands}"
       sim_gazebo="${sim_gazebo}"
       sim_ignition="${sim_ignition}"

File: scout/scout_description/urdf/kortex.ros2_control.xacro (robot description, xacro)
@@ -5,5 +5,5 @@
     prefix
     use_fake_hardware:=false
-    fake_sensor_commands:=false
+    mock_sensor_commands:=false
     sim_gazebo:=false
     sim_ignition:=false
@@ -39,5 +39,5 @@
         <xacro:if value="${use_fake_hardware}">
           <plugin>mock_components/GenericSystem</plugin>
-          <param name="fake_sensor_commands">${fake_sensor_commands}</param>
+          <param name="mock_sensor_commands">${mock_sensor_commands}</param>
           <param name="state_following_offset">0.0</param>
         </xacro:if>
@@ -64,5 +64,5 @@
         </command_interface>
         <state_interface name="position">
-          <param name="initial_value">${initial_positions['joint_1']}</param>
+          <param name="initial_value">${initial_positions['arm_joint_1']}</param>
         </state_interface>
         <state_interface name="velocity"/>
@@ -75,5 +75,5 @@
         </command_interface>
         <state_interface name="position">
-          <param name="initial_value">${initial_positions['joint_2']}</param>
+          <param name="initial_value">${initial_positions['arm_joint_2']}</param>
         </state_interface>
         <state_interface name="velocity"/>
@@ -86,5 +86,5 @@
         </command_interface>
         <state_interface name="position">
-          <param name="initial_value">${initial_positions['joint_3']}</param>
+          <param name="initial_value">${initial_positions['arm_joint_3']}</param>
         </state_interface>
         <state_interface name="velocity"/>
@@ -97,5 +97,5 @@
         </command_interface>
         <state_interface name="position">
-          <param name="initial_value">${initial_positions['joint_4']}</param>
+          <param name="initial_value">${initial_positions['arm_joint_4']}</param>
         </state_interface>
         <state_interface name="velocity"/>
@@ -108,5 +108,5 @@
         </command_interface>
         <state_interface name="position">
-          <param name="initial_value">${initial_positions['joint_5']}</param>
+          <param name="initial_value">${initial_positions['arm_joint_5']}</param>
         </state_interface>
         <state_interface name="velocity"/>
@@ -119,5 +119,5 @@
         </command_interface>
         <state_interface name="position">
-          <param name="initial_value">${initial_positions['joint_6']}</param>
+          <param name="initial_value">${initial_positions['arm_joint_6']}</param>
         </state_interface>
         <state_interface name="velocity"/>
@@ -130,5 +130,5 @@
         </command_interface>
         <state_interface name="position">
-          <param name="initial_value">${initial_positions['joint_7']}</param>
+          <param name="initial_value">${initial_positions['arm_joint_7']}</param>
         </state_interface>
         <state_interface name="velocity"/>

File: scout/scout_description/urdf/scout_kinova.xacro (robot description, xacro)
@@ -21,6 +21,6 @@
     <xacro:property name="gripper_joint_name" value="robotiq_2f_85_joint"/>
     <xacro:property name="use_fake_hardware" value="true" />
-    <xacro:property name="fake_sensor_commands" value="false" />
-    <xacro:property name="sim_gazebo" value="false" />
+    <xacro:property name="mock_sensor_commands" value="false" />
+    <xacro:property name="sim_gazebo" value="true" />
     <xacro:property name="sim_ignition" value="false" />
     <xacro:property name="sim_isaac" value="false" />
@@ -28,5 +28,5 @@
     <xacro:property name="isaac_joint_states" value="/isaac_joint_states" />
     <xacro:property name="use_external_cable" value="false" />
-    <xacro:property name="initial_positions" value="${dict(joint_1=0.0,joint_2=0.0,joint_3=0.0,joint_4=0.0,joint_5=0.0,joint_6=0.0,joint_7=0.0)}" />
+    <xacro:property name="initial_positions" value="${dict(arm_joint_1=0.0,arm_joint_2=0.0,arm_joint_3=0.0,arm_joint_4=0.0,arm_joint_5=0.0,arm_joint_6=0.0,arm_joint_7=0.0)}" />
     <xacro:include filename="$(find scout_description)/urdf/scout_wheel_type1.xacro" />
     <xacro:include filename="$(find scout_description)/urdf/scout_wheel_type2.xacro" />
@@ -121,5 +121,5 @@
         gripper_max_force="${gripper_max_force}"
         use_fake_hardware="${use_fake_hardware}"
-        fake_sensor_commands="${fake_sensor_commands}"
+        mock_sensor_commands="${mock_sensor_commands}"
         sim_gazebo="${sim_gazebo}"
         sim_ignition="${sim_ignition}"

Commit message: ignition migration attempt

File: scout/scout_description/urdf/gen3_macro.xacro (robot description, xacro)
@@ -8,5 +8,5 @@
     dof
     vision
-    prefix
+    prefix:=arm_
     *origin
     robot_ip

File: scout/scout_description/urdf/kortex.ros2_control.xacro (robot description, xacro)
@@ -13,5 +13,5 @@
     use_internal_bus_gripper_comm:=true
     tf_prefix
-    initial_positions:=${dict(joint_1=0.0,joint_2=0.0,joint_3=0.0,joint_4=0.0,joint_5=0.0,joint_6=0.0,joint_7=0.0)}
+    initial_positions:=${dict(arm_joint_1=0.0,arm_joint_2=0.0,arm_joint_3=0.0,arm_joint_4=0.0,arm_joint_5=0.0,arm_joint_6=0.0,arm_joint_7=0.0)}
     robot_ip
     username
@@ -30,5 +30,15 @@
         </xacro:if>
         <xacro:if value="${sim_ignition}">
-          <plugin>ign_ros2_control/IgnitionSystem</plugin>
+        <!-- Gazebo plugins -->
+          <gazebo reference="world">
+          </gazebo>
+          <gazebo>
+            <plugin filename="libign_ros2_control-system.so" name="ign_ros2_control::IgnitionROS2ControlPlugin">
+              <controller_manager_node_name>controller_manager</controller_manager_node_name>
+            </plugin>
+            <plugin filename="libignition-gazebo-sensors-system.so" name="ignition::gazebo::systems::Sensors">
+              <render_engine>ogre</render_engine>
+            </plugin>
+          </gazebo>
         </xacro:if>
         <xacro:if value="${sim_isaac}">

File: scout/scout_description/urdf/scout_kinova.xacro (robot description, xacro)
@@ -1,4 +1,4 @@
 <?xml version="1.0"?>
-<robot name="scout_v2" xmlns:xacro="http://ros.org/wiki/xacro">
+<robot name="scout_kinova" xmlns:xacro="http://ros.org/wiki/xacro">
     <!-- Define Properties -->
     <xacro:property name="robot_namespace" value="/" />
@@ -22,6 +22,6 @@
     <xacro:property name="use_fake_hardware" value="true" />
     <xacro:property name="mock_sensor_commands" value="false" />
-    <xacro:property name="sim_gazebo" value="true" />
-    <xacro:property name="sim_ignition" value="false" />
+    <xacro:property name="sim_gazebo" value="false" />
+    <xacro:property name="sim_ignition" value="true" />
     <xacro:property name="sim_isaac" value="false" />
     <xacro:property name="isaac_joint_commands" value="/isaac_joint_commands" />
